File: ntp-devboard.kicad_pcb (KiCad board)
At the start: 2 copper layers, 42.4 x 51 mm, 73 parts, among them J1 USB_C_Receptacle_USB2.0_14P, J2 Conn_01x07, J3 Conn_01x20, J4 Conn_01x04, J6 RJ45_Hanrun_HR911105A_Horizon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, SW1 SW_Push, U1 RP2040, U2 MCP1700x-330xxTT, U3 LAN9250/ML, U4 W25Q16JVUXIQ TR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

Commit message: bom optimisation
Parts:
- C37: footprint Capacitor_SMD:C_0402_1005Metric -> Capacitor_SMD:C_0805_2012Metric
- FB1, FB2, FB3, FB4: footprint Inductor_SMD:L_0201_0603Metric -> Inductor_SMD:L_0603_1608Metric
- R11, R12: value 330 -> 10K
- moved C38 4.80 mm to (137.9, 122.3)
- moved C37 2.75 mm to (144.8, 113.4), turned to 0 degrees
- moved FB1 1.97 mm to (138.8, 118.9)
- moved FB3 1.63 mm to (138.7, 120.5)
- moved FB2 0.79 mm to (138.8, 117.4)
- moved FB4 0.70 mm to (133.8, 118.8)
Routing:
- net +3V3: track 161.7 -> 163.3 mm
- net C34: track 35.6 -> 37.0 mm, vias 2 -> 3
- net C35: track 43.3 -> 42.1 mm
- net GND: track 80.4 -> 80.5 mm, vias 60 -> 57

Commit message: uhm, _minor_ mistake
Parts:
- added J5: Conn_01x02, Connector_PinHeader_2.54mm:PinHeader_1x02_P2.54mm_Vertical, F.Cu at (147.0, 96.3)
Connections:
- J6 pad 10: GND -> unconnected-(J6-Pad10)
- J6 pad 11: GND -> unconnected-(J6-Pad11)
- J6 pad 12: LAN46 -> unconnected-(J6-Pad12)
- J6 pad 9: LAN45 -> unconnected-(J6-Pad9)
Routing:
- net LAN46: track 28.2 -> 16.7 mm
- net LAN45: track 24.9 -> 14.7 mm

Commit message: cooked ah decoupling caps
Parts:
- C18, C19: value 33pF -> 15pF
- R15: value 12.1K -> 12K
- R3, R4: value 27 -> 22
- moved C24 23.2 mm to (145.3, 104.5), turned to 90 degrees
- moved C38 22.3 mm to (145.5, 101.3), turned to 0 degrees
- moved FB3 19.4 mm to (146.0, 102.5)
- moved C26 17.2 mm to (142.0, 108.0), turned to 0 degrees
- moved C27 14.0 mm to (141.6, 113.6), turned to -90 degrees
- moved FB2 11.4 mm to (127.6, 115.2), turned to 90 degrees
- moved FB1 11.2 mm to (127.6, 118.3), turned to 90 degrees
- moved C25 9.71 mm to (130.0, 109.5)
- moved C32 9.26 mm to (139.2, 117.1), turned to 180 degrees
- moved C33 7.25 mm to (126.8, 112.5), turned to 180 degrees
- moved C28 6.19 mm to (134.0, 117.5), turned to -90 degrees
- moved FB4 2.71 mm to (133.6, 121.5)
- moved C29 1.91 mm to (129.9, 114.5)
- moved R16 1.56 mm to (128.9, 108.4)
- moved C21 1.05 mm to (129.3, 119.2)
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Routing:
- net GND: track 80.5 -> 102.3 mm, vias 57 -> 65
- net C34: track 37.0 -> 42.3 mm
- net C40: track 45.6 -> 48.5 mm, vias 2 -> 5
- net +3V3: track 163.3 -> 165.9 mm, vias 4 -> 6
- net C35: track 42.1 -> 39.8 mm
- net OSOUT: track 4.61 -> 6.08 mm
- net Net-(U3-OSCVSS): track 1.20 -> 2.55 mm
- net Net-(U3-FXLOSEN): track 4.33 -> 3.27 mm

Commit message: powertraces go brr
Routing:
- net GND: track 102.3 -> 102.4 mm, vias 65 -> 105

Commit message: update sch and pcb
Parts:
- moved FB1 21.6 mm to (145.7, 106.5), turned to 180 degrees
- moved C21 11.0 mm to (140.3, 118.1)
- moved FB2 8.90 mm to (128.0, 106.3), turned to 0 degrees
- moved FB4 4.99 mm to (137.4, 118.3)
- moved R11 4.24 mm to (131.4, 118.0)
- moved C31 3.11 mm to (128.4, 114.3), turned to -90 degrees
- moved C20 2.38 mm to (129.9, 118.6), turned to 90 degrees
- moved Y2 0.50 mm to (124.4, 107.2)
- turned R13 to 0 degrees
Connections:
- net C34 renamed Power_Lan
- net C35 renamed POWER_LAN12
- net C40 renamed TXRX_POWER
- R13 pad 1: Net-(U3-FXLOSEN) -> GND
- R13 pad 2: GND -> Net-(U3-FXLOSEN)
Routing:
- net TXRX_POWER: track 48.8 -> 35.3 mm, vias 5 -> 4
- net GND: track 102.4 -> 90.0 mm, vias 105 -> 233
- net POWER_LAN12: track 39.8 -> 30.6 mm, vias 2 -> 4
- net TX+: track 12.3 -> 5.92 mm
- net +3V3: track 166.1 -> 159.7 mm, vias 6 -> 40
- net GPIO5: track 29.3 -> 23.4 mm
- net TX-: track 12.4 -> 7.73 mm
- net Power_Lan: track 42.3 -> 38.4 mm
- net RX-: track 9.04 -> 7.64 mm
- net OSIN: track 7.67 -> 8.70 mm, vias 0 -> 2
- net RX+: track 9.08 -> 9.76 mm
- net Net-(C19-Pad2): track 4.27 -> 4.78 mm
- net (no net): vias 0 -> 5
- added copper zone on In2.Cu, net +3V3
- added copper zone on In1.Cu, net GND
Other:
- copper layers 2 -> 4
